Commit message: feat(gripper): 统一夹爪为单一 gripper 关节（0–0.1 m）
- agx_arm_urdf：新增 gripper 主关节，gripper_joint1/2 改为 mimic 从动关节。
- agx_arm_ctrl：移除 publish_gripper_joint，JointState 仅发布/接收 gripper。
- agx_arm_moveit：控制器、SRDF、ros2_control 仅控制 gripper；joint1/2 标为 passive。
- 更新 README / README_EN / agx_arm_moveit 文档。

---

feat(gripper): unify gripper on a single 0–0.1 m joint

- agx_arm_urdf: add master gripper joint; drive gripper_joint1/2 via mimic.
- agx_arm_ctrl: drop publish_gripper_joint; publish/control gripper only in JointState.
- agx_arm_moveit: control gripper only in controllers, SRDF, and ros2_control; mark joint1/2 passive.
- Update README / README_EN / agx_arm_moveit docs.

File: src/agx_arm_moveit/config/agx_arm.ros2_control.xacro (robot description, xacro)
@@ -59,15 +59,8 @@
       </xacro:if>
       <xacro:if value="${effector_type == 'agx_gripper'}">
-        <joint name="gripper_joint1">
+        <joint name="gripper">
           <command_interface name="position" />
           <state_interface name="position">
-            <param name="initial_value">${initial_positions['gripper_joint1']}</param>
-          </state_interface>
-          <state_interface name="velocity" />
-        </joint>
-        <joint name="gripper_joint2">
-          <command_interface name="position" />
-          <state_interface name="position">
-            <param name="initial_value">${initial_positions['gripper_joint2']}</param>
+            <param name="initial_value">${initial_positions['gripper']}</param>
           </state_interface>
           <state_interface name="velocity" />

File: src/agx_arm_moveit/config/agx_arm.srdf.xacro (robot description, xacro)
@@ -16,19 +16,17 @@
       <link name="gripper_link1" />
       <link name="gripper_link2" />
-      <joint name="gripper_joint1" />
-      <joint name="gripper_joint2" />
+      <joint name="gripper" />
     </group>
+    <passive_joint name="gripper_joint1" />
+    <passive_joint name="gripper_joint2" />
     <end_effector name="gripper_eef" parent_link="tcp_link" group="gripper" parent_group="arm" />
     <group_state name="gripper_open" group="gripper">
-      <joint name="gripper_joint1" value="0.05" />
-      <joint name="gripper_joint2" value="-0.05" />
+      <joint name="gripper" value="0.1" />
     </group_state>
     <group_state name="gripper_half" group="gripper">
-      <joint name="gripper_joint1" value="0.025" />
-      <joint name="gripper_joint2" value="-0.025" />
+      <joint name="gripper" value="0.05" />
     </group_state>
     <group_state name="gripper_close" group="gripper">
-      <joint name="gripper_joint1" value="0.0" />
-      <joint name="gripper_joint2" value="0.0" />
+      <joint name="gripper" value="0.0" />
     </group_state>
     <disable_collisions link1="gripper_base" link2="${flange_link}" reason="Adjacent" />
