Commit message: feat(moveit): 调整机械臂初始姿态

File: src/agx_arm_moveit/config/agx_arm.srdf.xacro (robot description, xacro)
@@ -341,5 +341,5 @@
     <group_state name="home" group="arm">
       <joint name="joint1" value="0" />
-      <joint name="joint2" value="0" />
+      <joint name="joint2" value="1.3962634016" />
       <joint name="joint3" value="0" />
       <joint name="joint4" value="0" />
@@ -351,5 +351,5 @@
     <group_state name="home" group="arm">
       <joint name="joint1" value="0" />
-      <joint name="joint2" value="0" />
+      <joint name="joint2" value="1.3962634016" />
       <joint name="joint3" value="0" />
       <joint name="joint4" value="0" />
